File: hardware/Hardware_Rev1.kicad_pcb (KiCad board)
At the start: 2 copper layers, 123.2 x 45.5 mm, 56 parts, among them J1 RJ45_LED_Shielded, J2 6P6C, Q1 BUK9M9R5-40HX, Q2 BUK9M9R5-40HX, Q3 BUK9M9R5-40HX, U1 LT1910, U2 LT1910, U3 OKI, U4 LT1910, U5 TSR_1-2450, U6 Teensy4.1_DEV-16771

Commit message: good progress on traces, finishing them tomorrow probably
Parts:
- moved D5 3.30 mm to (99.2, 69.8)
- moved C3 3.30 mm to (102.9, 66.8)
- moved D1 3.30 mm to (99.2, 68.3)
- moved R3 3.30 mm to (102.9, 68.3)
- moved R8 3.30 mm to (102.9, 69.8)
- moved V4 2.61 mm to (201.0, 88.3)
- moved V3 2.51 mm to (201.0, 58.7)
- moved U6 2.29 mm to (228.1, 114.0)
- moved J2 1.78 mm to (142.9, 87.7)
- moved C13 1.78 mm to (130.9, 88.7)
- moved J1 1.78 mm to (136.9, 62.7)
- moved C6 1.52 mm to (123.4, 67.3)
- moved C7 1.52 mm to (123.4, 68.8)
- moved D4 1.52 mm to (127.0, 70.4)
- moved R6 1.52 mm to (123.4, 70.4)
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Routing:
- net +3V3: track 16.5 -> 257.9 mm, vias 0 -> 2
- net Heater2: track 2.76 -> 27.3 mm
- net Heater1: track 3.27 -> 20.4 mm
- net Net-(R11-Pad2): track 0.00 -> 12.7 mm
- net Net-(R10-Pad2): track 0.00 -> 12.3 mm
- net Net-(Conn4-Pad1): track 0.00 -> 11.8 mm, vias 0 -> 1
- net Net-(R12-Pad2): track 0.00 -> 5.31 mm
- net Net-(D3-Pad2): track 0.00 -> 1.76 mm
Other:
- board size 123.2 x 45.5 mm -> 120.7 x 45.5 mm
- board text added: "1"
- board text added: "2"
- board text added: "3"
- board text added: "Water Heater Board 2022 - Rev 1 Mars Rover Design Team Missouri S&T, 2022 Jacob Byers, James Elverson, Joshua Perkins"
- board text removed: "Label These :)"
- board text removed: "Water Heater Board 2022 - Rev 1 Jacob Byers, James Elverson, Joshua Perkins #ROVESOHARD"

Commit message: IUY
Routing:
- net Net-(Conn6-Pad1): track 0.00 -> 20.6 mm, vias 0 -> 1
- net Net-(Conn10-Pad1): track 0.00 -> 19.4 mm, vias 0 -> 1
- net Net-(Q2-Pad4): track 0.00 -> 16.3 mm, vias 0 -> 2
- net Heater3: track 3.02 -> 19.0 mm
- net Net-(Q3-Pad4): track 0.00 -> 15.8 mm, vias 0 -> 2
- net Net-(Conn4-Pad1): track 11.8 -> 21.6 mm
Changed lines of the file:
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@@
   (segment (start 140.208 79.248) (end 140.208 82.804) (width 0.254) (layer "B.Cu") (net 8))
   (segment (start 140.208 83.312) (end 141.478 84.582) (width 0.254) (layer "B.Cu") (net 8))
-  (segment (start 125.659 56.317) (end 125.73 56.388) (width 1.397) (layer "F.Cu") (net 11))
-  (segment (start 125.659 55.129) (end 125.659 56.317) (width 1.397) (layer "F.Cu") (net 11))
-  (via (at 125.73 56.388) (size 0.8) (drill 0.4) (layers "F.Cu" "B.Cu") (net 11))
-  (segment (start 131.064 58.166) (end 131.3053 58.166) (width 1.397) (layer "B.Cu") (net 11))
-  (segment (start 129.6892 56.7912) (end 131.064 58.166) (width 1.397) (layer "B.Cu") (net 11))
-  (segment (start 131.3053 58.166) (end 131.8133 58.674) (width 1.397) (layer "B.Cu") (net 11))
-  (segment (start 128.4192 56.7912) (end 129.6892 56.7912) (width 1.397) (layer "B.Cu") (net 11))
-  (segment (start 125.4633 56.388) (end 123.1773 58.674) (width 1.397) (layer "B.Cu") (net 11))
-  (segment (start 128.016 56.388) (end 128.4192 56.7912) (width 1.397) (layer "B.Cu") (net 11))
-  (segment (start 125.73 56.388) (end 128.016 56.388) (width 1.397) (layer "B.Cu") (net 11))
-  (segment (start 125.73 56.388) (end 125.4633 56.388) (width 1.397) (layer "B.Cu") (net 11))
+  (segment (start 125.659 57.841) (end 125.73 57.912) (width 1.524) (layer "F.Cu") (net 11))
+  (segment (start 127.5975 60.706) (end 125.73 58.8385) (width 0.254) (layer "F.Cu") (net 11))
+  (segment (start 125.659 55.129) (end 125.659 57.841) (width 1.524) (layer "F.Cu") (net 11))
+  (segment (start 125.73 58.8385) (end 125.73 57.912) (width 0.254) (layer "F.Cu") (net 11))
+  (via (at 125.73 57.912) (size 0.8) (drill 0.4) (layers "F.Cu" "B.Cu") (net 11))
+  (segment (start 125.73 59.69) (end 124.46 60.96) (width 1.524) (layer "B.Cu") (net 11))
+  (segment (start 125.73 57.912) (end 125.73 59.69) (width 1.524) (layer "B.Cu") (net 11))
+  (segment (start 125.73 57.912) (end 125.73 58.42) (width 1.524) (layer "B.Cu") (net 11))
+  (segment (start 129.7813 60.706) (end 131.8133 58.674) (width 1.524) (layer "B.Cu") (net 11))
+  (segment (start 123.698 60.96) (end 123.1773 60.4393) (width 1.524) (layer "B.Cu") (net 11))
+  (segment (start 123.1773 60.4393) (end 123.1773 58.674) (width 1.524) (layer "B.Cu") (net 11))
+  (segment (start 128.016 60.706) (end 129.7813 60.706) (width 1.524) (layer "B.Cu") (net 11))
+  (segment (start 124.46 60.96) (end 123.698 60.96) (width 1.524) (layer "B.Cu") (net 11))
+  (segment (start 125.73 58.42) (end 128.016 60.706) (width 1.524) (layer "B.Cu") (net 11))
+  (segment (start 169.347 57.587) (end 169.418 57.658) (width 1.524) (layer "F.Cu") (net 12))
+  (segment (start 169.418 58.8245) (end 169.418 57.658) (width 0.254) (layer "F.Cu") (net 12))
+  (segment (start 169.347 55.026) (end 169.347 57.587) (width 1.524) (layer "F.Cu") (net 12))
+  (segment (start 171.2995 60.706) (end 169.418 58.8245) (width 0.254) (layer "F.Cu") (net 12))
+  (via (at 169.418 57.658) (size 0.8) (drill 0.4) (layers "F.Cu" "B.Cu") (net 12))
+  (segment (start 169.418 59.944) (end 169.926 60.452) (width 1.524) (layer "B.Cu") (net 12))
+  (segment (start 168.91 60.452) (end 167.386 60.452) (width 1.524) (layer "B.Cu") (net 12))
+  (segment (start 169.418 59.944) (end 168.91 60.452) (width 1.524) (layer "B.Cu") (net 12))
+  (segment (start 175.514 59.69) (end 175.514 58.674) (width 1.524) (layer "B.Cu") (net 12))
+  (segment (start 174.752 60.452) (end 175.514 59.69) (width 1.524) (layer "B.Cu") (net 12))
+  (segment (start 167.386 60.452) (end 166.8653 59.9313) (width 1.524) (layer "B.Cu") (net 12))
+  (segment (start 169.926 60.452) (end 174.752 60.452) (width 1.524) (layer "B.Cu") (net 12))
+  (segment (start 166.8653 59.9313) (end 166.8653 58.674) (width 1.524) (layer "B.Cu") (net 12))
+  (segment (start 169.418 57.658) (end 169.418 59.944) (width 1.524) (layer "B.Cu") (net 12))
+  (segment (start 147.574 58.8245) (end 147.574 57.658) (width 0.254) (layer "F.Cu") (net 14))
+  (segment (start 147.503 57.587) (end 147.574 57.658) (width 1.524) (layer "F.Cu") (net 14))
+  (segment (start 147.503 55.637) (end 147.503 57.587) (width 1.524) (layer "F.Cu") (net 14))
+  (segment (start 149.4555 60.706) (end 147.574 58.8245) (width 0.254) (layer "F.Cu") (net 14))
+  (via (at 147.574 57.658) (size 0.8) (drill 0.4) (layers "F.Cu" "B.Cu") (net 14))
+  (segment (start 147.574 59.944) (end 147.066 60.452) (width 1.524) (layer "B.Cu") (net 14))
+  (segment (start 147.066 60.452) (end 145.542 60.452) (width 1.524) (layer "B.Cu") (net 14))
+  (segment (start 151.892 60.452) (end 153.67 58.674) (width 1.524) (layer "B.Cu") (net 14))
+  (segment (start 147.574 59.944) (end 148.082 60.452) (width 1.524) (layer "B.Cu") (net 14))
+  (segment (start 148.082 60.452) (end 151.892 60.452) (width 1.524) (layer "B.Cu") (net 14))
+  (segment (start 145.542 60.452) (end 145.0378 59.9478) (width 1.524) (layer "B.Cu") (net 14))
+  (segment (start 145.0378 59.9478) (end 145.0378 58.674) (width 1.524) (layer "B.Cu") (net 14))
+  (segment (start 147.574 57.658) (end 147.574 59.944) (width 1.524) (layer "B.Cu") (net 14))
   (segment (start 101.9575 68.326) (end 100.048 68.326) (width 0.254) (layer "F.Cu") (net 15))
   (segment (start 129.4225 60.706) (end 131.064 60.706) (width 0.254) (layer "F.Cu") (net 16))
@@
   (segment (start 136.906 56.388) (end 133.858 56.388) (width 0.254) (layer "B.Cu") (net 32))
   (segment (start 139.7 53.594) (end 136.906 56.388) (width 0.254) (layer "B.Cu") (net 32))
+  (segment (start 172.72 56.642) (end 171.104 55.026) (width 0.254) (layer "F.Cu") (net 33))
+  (segment (start 182.499 52.959) (end 183.388 53.848) (width 0.254) (layer "F.Cu") (net 33))
+  (segment (start 182.499 52.672) (end 182.499 52.959) (width 0.254) (layer "F.Cu") (net 33))
+  (segment (start 171.104 55.026) (end 170.647 55.026) (width 0.254) (layer "F.Cu") (net 33))
+  (via (at 183.388 53.848) (size 0.8) (drill 0.4) (layers "F.Cu" "B.Cu") (net 33))
+  (via (at 172.72 56.642) (size 0.8) (drill 0.4) (layers "F.Cu" "B.Cu") (net 33))
+  (segment (start 180.848 56.642) (end 172.72 56.642) (width 0.254) (layer "B.Cu") (net 33))
+  (segment (start 183.388 54.102) (end 180.848 56.642) (width 0.254) (layer "B.Cu") (net 33))
+  (segment (start 183.388 53.848) (end 183.388 54.102) (width 0.254) (layer "B.Cu") (net 33))
+  (segment (start 160.655 52.959) (end 161.544 53.848) (width 0.254) (layer "F.Cu") (net 34))
+  (segment (start 151.13 56.642) (end 150.125 55.637) (width 0.254) (layer "F.Cu") (net 34))
+  (segment (start 150.125 55.637) (end 148.803 55.637) (width 0.254) (layer "F.Cu") (net 34))
+  (segment (start 160.655 52.926) (end 160.655 52.959) (width 0.254) (layer "F.Cu") (net 34))
+  (via (at 161.544 53.848) (size 0.8) (drill 0.4) (layers "F.Cu" "B.Cu") (net 34))
+  (via (at 151.13 56.642) (size 0.8) (drill 0.4) (layers "F.Cu" "B.Cu") (net 34))
+  (segment (start 159.004 56.642) (end 151.13 56.642) (width 0.254) (layer "B.Cu") (net 34))
+  (segment (start 161.544 54.102) (end 159.004 56.642) (width 0.254) (layer "B.Cu") (net 34))
+  (segment (start 161.544 53.848) (end 161.544 54.102) (width 0.254) (layer "B.Cu") (net 34))
   (segment (start 137.414 59.7935) (end 137.414 57.945) (width 0.254) (layer "F.Cu") (net 36))
   (segment (start 137.414 57.945) (end 137.287 57.818) (width 0.254) (layer "F.Cu") (net 36))
@@
   (segment (start 187.706 66.1905) (end 187.706 69.342) (width 0.254) (layer "F.Cu") (net 41))
   (segment (start 187.706 69.342) (end 186.182 70.866) (width 0.254) (layer "F.Cu") (net 41))
+  (segment (start 138.811 60.833) (end 142.24 64.262) (width 0.254) (layer "F.Cu") (net 42))
   (segment (start 138.811 57.818) (end 138.811 60.833) (width 0.254) (layer "F.Cu") (net 42))
+  (segment (start 145.796 64.262) (end 148.082 66.548) (width 0.254) (layer "F.Cu") (net 42))
+  (segment (start 148.082 66.548) (end 148.082 70.866) (width 0.254) (layer "F.Cu") (net 42))
+  (segment (start 142.24 64.262) (end 145.796 64.262) (width 0.254) (layer "F.Cu") (net 42))
   (segment (start 182.499 64.643) (end 185.166 67.31) (width 0.254) (layer "F.Cu") (net 43))
   (segment (start 185.674 73.152) (end 186.436 73.152) (width 0.254) (layer "F.Cu") (net 43))

Commit message: made layout changes, didn't finish everything tho
Parts:
- moved U6 154.7 mm to (90.2, 43.9), turned to 0 degrees
- moved J1 75.6 mm to (211.1, 77.5), turned to 90 degrees
- moved C13 56.7 mm to (185.1, 72.0), turned to 0 degrees
- moved J2 43.4 mm to (186.1, 83.9), turned to 180 degrees
- moved D7 32.6 mm to (179.9, 91.2), turned to 180 degrees
- moved R10 31.2 mm to (176.4, 91.2), turned to 180 degrees
- moved D8 29.8 mm to (179.9, 89.4), turned to 180 degrees
- moved R11 28.0 mm to (176.4, 89.4), turned to 180 degrees
- moved D9 27.1 mm to (179.8, 87.6), turned to 180 degrees
- moved R12 25.1 mm to (176.3, 87.6), turned to 180 degrees
- moved Conn3 21.4 mm to (209.1, 65.5), turned to -90 degrees
- moved U3 13.0 mm to (100.1, 68.6)
- moved C6 12.4 mm to (111.1, 66.3)
- moved C7 12.4 mm to (111.1, 67.8)
- moved D4 12.4 mm to (114.7, 69.3)
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Routing:
- net +3V3: track 257.9 -> 0.61 mm, vias 2 -> 0
- net Heater2: track 27.3 -> 2.76 mm
- net Heater3: track 19.0 -> 3.02 mm
- net Heater1: track 20.4 -> 6.57 mm
- net Net-(R11-Pad2): track 12.7 -> 1.99 mm
- net Net-(R10-Pad2): track 12.3 -> 1.73 mm
- net +12V: track 9.51 -> 0.00 mm
- net Net-(R12-Pad2): track 5.31 -> 1.88 mm
- removed copper zone on F.Cu, net +12V
Other:
- board size 120.7 x 45.5 mm -> 120.7 x 44.5 mm

Commit message: maor
Parts:
- moved R10 62.1 mm to (114.3, 90.4), turned to 90 degrees
- moved R11 59.5 mm to (116.8, 90.4), turned to 90 degrees
- moved R12 44.3 mm to (132.1, 90.4), turned to 90 degrees
- moved D8 37.5 mm to (142.5, 91.4)
- moved D9 37.4 mm to (142.5, 89.7)
- moved D7 37.4 mm to (142.6, 93.2)
- moved Q1 12.0 mm to (126.0, 65.6), turned to -90 degrees
- moved J1 8.90 mm to (202.2, 77.9)
- moved Conn3 8.89 mm to (200.2, 65.5)
- moved C13 8.89 mm to (176.2, 72.0)
- moved J2 8.89 mm to (177.2, 83.9)
- moved V4 8.82 mm to (192.2, 86.8)
- moved V3 8.81 mm to (192.2, 58.7)
- moved V1 0.59 mm to (96.3, 86.7)
- moved R1 0.51 mm to (137.9, 60.7)
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Routing:
- net Net-(Conn4-Pad1): track 21.6 -> 0.00 mm, vias 1 -> 0
- net Net-(Q1-Pad4): track 16.4 -> 0.00 mm, vias 2 -> 0
- net Heater3: track 3.02 -> 0.00 mm
- net Net-(C1-Pad1): track 2.08 -> 0.00 mm
- net Net-(R1-Pad2): track 2.03 -> 0.00 mm
- net Net-(R11-Pad2): track 1.99 -> 0.00 mm
- net Net-(R12-Pad2): track 1.88 -> 0.00 mm
- net Net-(D8-Pad2): track 1.78 -> 0.00 mm
- net Net-(D9-Pad2): track 1.77 -> 0.00 mm
- net Net-(D7-Pad2): track 1.77 -> 0.00 mm
- net Net-(R10-Pad2): track 1.73 -> 0.00 mm
Other:
- board size 120.7 x 44.5 mm -> 111.8 x 44 mm

Commit message: closing kicad
Parts:
- moved D7 43.9 mm to (186.5, 93.5)
- moved D8 43.9 mm to (186.4, 91.7)
- moved D9 43.9 mm to (186.4, 89.9)
Routing:
- net Temp2: track 0.00 -> 46.3 mm, vias 0 -> 1
Other:
- outline, holes or cut-outs redrawn
Changed lines of the file:
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@@
   )
   (footprint "LED_SMD:LED_0603_1608Metric_Pad1.05x0.95mm_HandSolder" (layer "F.Cu")
-    (at 142.494 89.662 180)
+    (at 186.436 89.916 180)
     (descr "LED SMD 0603 (1608 Metric), square (rectangular) end terminal, IPC_7351 nominal, (Body size source: http://www.tortai-tech.com/upload/download/2011102023233369053.pdf), generated with kicad-footprint-generator")
     (tags "LED handsolder")
@@
   )
   (footprint "LED_SMD:LED_0603_1608Metric_Pad1.05x0.95mm_HandSolder" (layer "F.Cu")
-    (at 142.607 93.218 180)
+    (at 186.549 93.472 180)
     (descr "LED SMD 0603 (1608 Metric), square (rectangular) end terminal, IPC_7351 nominal, (Body size source: http://www.tortai-tech.com/upload/download/2011102023233369053.pdf), generated with kicad-footprint-generator")
     (tags "LED handsolder")
@@
   )
   (footprint "LED_SMD:LED_0603_1608Metric_Pad1.05x0.95mm_HandSolder" (layer "F.Cu")
-    (at 142.494 91.44 180)
+    (at 186.436 91.694 180)
     (descr "LED SMD 0603 (1608 Metric), square (rectangular) end terminal, IPC_7351 nominal, (Body size source: http://www.tortai-tech.com/upload/download/2011102023233369053.pdf), generated with kicad-footprint-generator")
     (tags "LED handsolder")
@@
   (gr_line (start 200.152 85.852) (end 200.152 89.408) (layer "Edge.Cuts") (width 0.05))
   (gr_line (start 88.392 59.436) (end 88.392 69.85) (layer "Edge.Cuts") (width 0.05))
+  (gr_line (start 194.31 94.736713) (end 195.828713 94.736713) (layer "Edge.Cuts") (width 0.05))
+  (gr_line (start 155.702 94.742) (end 175.514 94.742) (layer "Edge.Cuts") (width 0.05))
   (gr_line (start 194.31 50.8) (end 196.008327 50.752682) (layer "Edge.Cuts") (width 0.05))
   (gr_arc (start 92.456 94.742) (mid 89.582318 93.551682) (end 88.392 90.678) (layer "Edge.Cuts") (width 0.05))
@@
   (gr_line (start 98.806 50.8) (end 178.816 50.8) (layer "Edge.Cuts") (width 0.05))
   (gr_line (start 88.392 54.864) (end 88.392 59.436) (layer "Edge.Cuts") (width 0.05))
+  (gr_line (start 189.992 94.742) (end 194.31 94.736713) (layer "Edge.Cuts") (width 0.05))
   (gr_line (start 88.392 82.55) (end 88.392 89.154) (layer "Edge.Cuts") (width 0.05))
   (gr_line (start 200.152 56.388) (end 200.072327 54.816682) (layer "Edge.Cuts") (width 0.05))
   (gr_line (start 200.152 58.674) (end 200.152 85.852) (layer "Edge.Cuts") (width 0.05))
   (gr_line (start 92.4814 50.7746) (end 98.806 50.8) (layer "Edge.Cuts") (width 0.05))
+  (gr_line (start 139.446 94.742) (end 155.702 94.742) (layer "Edge.Cuts") (width 0.05))
   (gr_arc (start 88.392 54.864) (mid 89.589758 51.972358) (end 92.4814 50.7746) (layer "Edge.Cuts") (width 0.05))
   (gr_line (start 88.392 76.454) (end 88.392 82.55) (layer "Edge.Cuts") (width 0.05))
   (gr_line (start 200.152 58.674) (end 200.152 56.388) (layer "Edge.Cuts") (width 0.05))
   (gr_line (start 88.392 69.85) (end 88.392 76.454) (layer "Edge.Cuts") (width 0.05))
+  (gr_line (start 175.514 94.742) (end 189.992 94.742) (layer "Edge.Cuts") (width 0.05))
   (gr_line (start 178.816 50.8) (end 194.31 50.8) (layer "Edge.Cuts") (width 0.05))
   (gr_line (start 88.392 89.154) (end 88.392 90.678) (layer "Edge.Cuts") (width 0.05))
@@
     (effects (font (size 1.5 1.5) (thickness 0.3)) (justify mirror))
   )
-  (gr_text "3" (at 146.812 93.218) (layer "F.SilkS")
+  (gr_text "3" (at 190.754 93.472) (layer "F.SilkS")
     (effects (font (size 1.246 1.246) (thickness 0.3)))
   )
@@
     (effects (font (size 1.246 1.246) (thickness 0.248)))
   )
-  (gr_text "1" (at 146.812 89.662) (layer "F.SilkS")
+  (gr_text "1" (at 190.754 89.916) (layer "F.SilkS")
     (effects (font (size 1.246 1.246) (thickness 0.3)))
   )
-  (gr_text "2" (at 146.812 91.44) (layer "F.SilkS")
+  (gr_text "2" (at 190.754 91.694) (layer "F.SilkS")
     (effects (font (size 1.246 1.246) (thickness 0.3)))
   )
@@
   (segment (start 166.8653 59.9313) (end 166.8653 58.674) (width 1.524) (layer "B.Cu") (net 12))
   (segment (start 169.418 57.658) (end 169.418 59.944) (width 1.524) (layer "B.Cu") (net 12))
+  (segment (start 122.936 70.104) (end 137.922 70.104) (width 0.254) (layer "F.Cu") (net 13))
+  (segment (start 137.922 70.104) (end 139.7 71.882) (width 0.254) (layer "F.Cu") (net 13))
+  (via (at 122.936 70.104) (size 0.8) (drill 0.4) (layers "F.Cu" "B.Cu") (net 13))
+  (segment (start 99.03037 70.104) (end 122.936 70.104) (width 0.254) (layer "B.Cu") (net 13))
+  (segment (start 96.298 67.37163) (end 99.03037 70.104) (width 0.254) (layer "B.Cu") (net 13))
+  (segment (start 96.298 66.294) (end 96.298 67.37163) (width 0.254) (layer "B.Cu") (net 13))
   (segment (start 147.574 58.8245) (end 147.574 57.658) (width 0.254) (layer "F.Cu") (net 14))
   (segment (start 147.503 57.587) (end 147.574 57.658) (width 1.524) (layer "F.Cu") (net 14))

Commit message: Added Image to silkscreen
WHAT IS MY PURPOSE
Parts:
- added G***: LOGO, LOGO, B.Cu at (45.7, 66.0)

Commit message: Spaced Out stuff
resistors and caps :)
Parts:
- moved Q3 12.0 mm to (146.8, 66.0), turned to -90 degrees
- moved C6 2.29 mm to (111.1, 64.0)
- moved R7 2.05 mm to (160.5, 63.0)
- moved R1 1.93 mm to (138.7, 62.5)
- moved C1 1.85 mm to (135.6, 62.5)
- moved R2 1.83 mm to (182.4, 62.5)
- moved R11 1.83 mm to (117.9, 91.9)
- moved C7 1.78 mm to (111.1, 66.0)
- moved C8 1.75 mm to (157.5, 63.0)
- moved C2 1.61 mm to (179.3, 62.5)
- moved R10 1.52 mm to (114.3, 91.9)
- moved R12 1.52 mm to (132.1, 91.9)
- moved D4 1.43 mm to (115.3, 68.1)
- moved R6 1.27 mm to (111.1, 68.1)
Routing:
- net Heater1: track 6.57 -> 0.00 mm
- net Net-(Conn10-Pad1): track 19.4 -> 15.9 mm
- net Net-(D4-Pad2): track 1.78 -> 0.00 mm
- net +3V3: track 0.61 -> 0.00 mm
