File: hardware/_autosave-Hardware_Rev1.kicad_pcb (KiCad board)
At the start: 2 copper layers, 111.8 x 44 mm, 57 parts, among them J1 RJ45_LED_Shielded, J2 6P6C, Q1 BUK9M9R5-40HX, Q2 BUK9M9R5-40HX, Q3 BUK9M9R5-40HX, U1 LT1910, U2 LT1910, U3 OKI, U4 LT1910, U5 TSR_1-2450, U6 Teensy4.1_DEV-16771

Commit message: lots of wires
dont roast pls
Routing:
- net +3V3: track 112.5 -> 124.5 mm, vias 3 -> 4
- net (no net): vias 0 -> 1
Changed lines of the file:
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@@
     (style (thickness 0.05) (arrow_length 1.27) (text_position_mode 0) (extension_height 0.58642) (extension_offset 0.5) keep_text_aligned)
   )
+  (via (at 123.952 81.28) (size 0.8) (drill 0.4) (layers "F.Cu" "B.Cu") (free) (net 0))
   (segment (start 179.324 63.3465) (end 178.1545 63.3465) (width 0.635) (layer "F.Cu") (net 2))
   (segment (start 154.658 62.202) (end 154.658 60.706) (width 0.635) (layer "F.Cu") (net 2))
@@
   (segment (start 100.076 68.58) (end 100.076 77.724) (width 1.27) (layer "B.Cu") (net 4))
   (segment (start 105.664 63.5) (end 105.664 68.072) (width 0.762) (layer "F.Cu") (net 5))
+  (segment (start 110.236 64.008) (end 110.236 68.022) (width 0.635) (layer "F.Cu") (net 5))
   (segment (start 105.664 68.072) (end 105.156 68.58) (width 0.762) (layer "F.Cu") (net 5))
   (segment (start 97.536 76.2) (end 96.266 76.2) (width 0.762) (layer "F.Cu") (net 5))
   (segment (start 175.646752 68.072) (end 161.676752 82.042) (width 0.635) (layer "F.Cu") (net 5))
   (segment (start 116.84 73.628554) (end 116.84 71.882) (width 0.762) (layer "F.Cu") (net 5))
+  (segment (start 122.428 79.216554) (end 122.428 79.248) (width 0.762) (layer "F.Cu") (net 5))
   (segment (start 188.468 66.04) (end 184.912 66.04) (width 0.635) (layer "F.Cu") (net 5))
   (segment (start 181.864 68.072) (end 175.646752 68.072) (width 0.635) (layer "F.Cu") (net 5))
@@
   (segment (start 114.268554 76.2) (end 116.84 73.628554) (width 0.762) (layer "F.Cu") (net 5))
   (segment (start 152.4 82.042) (end 147.32 87.122) (width 0.635) (layer "F.Cu") (net 5))
+  (segment (start 110.236 68.022) (end 110.186 68.072) (width 0.635) (layer "F.Cu") (net 5))
   (segment (start 193.202132 62.157) (end 192.351 62.157) (width 0.635) (layer "F.Cu") (net 5))
   (segment (start 199.168 62.484) (end 198.841 62.157) (width 0.635) (layer "F.Cu") (net 5))
   (segment (start 198.841 62.157) (end 193.202132 62.157) (width 0.635) (layer "F.Cu") (net 5))
+  (segment (start 116.84 73.628554) (end 122.428 79.216554) (width 0.762) (layer "F.Cu") (net 5))
   (segment (start 192.351 62.157) (end 188.468 66.04) (width 0.635) (layer "F.Cu") (net 5))
   (segment (start 161.676752 82.042) (end 157.48 82.042) (width 0.635) (layer "F.Cu") (net 5))
@@
   (via (at 105.664 63.5) (size 0.8) (drill 0.4) (layers "F.Cu" "B.Cu") (net 5))
   (via (at 184.912 66.04) (size 0.8) (drill 0.4) (layers "F.Cu" "B.Cu") (net 5))
+  (via (at 122.428 79.248) (size 0.8) (drill 0.4) (layers "F.Cu" "B.Cu") (net 5))
   (via (at 181.864 68.072) (size 0.8) (drill 0.4) (layers "F.Cu" "B.Cu") (net 5))
   (segment (start 105.41 63.246) (end 105.664 63.5) (width 0.762) (layer "B.Cu") (net 5))
