File: hardware/Hardware_Rev1.kicad_sch (KiCad schematic)
At the start: 134 parts, among them J1 RJ45_LED_Shielded, J2 6P6C, U3 OKI, U5 TSR_1-2450, U6 Teensy4.1_DEV-16771

Commit message: done with schematic ?
Parts:
- removed D7, D8, D9: LED(R), LED_SMD:LED_0603_1608Metric_Pad1.05x0.95mm_HandSolder, symbol Device:LED
- removed R10, R11, R12: 120, Resistor_SMD:R_0603_1608Metric_Pad0.98x0.95mm_HandSolder, symbol Device:R
- added D? (x11): LED(R), LED_SMD:LED_0603_1608Metric_Pad1.05x0.95mm_HandSolder, symbol Device:LED
- added R? (x11): 120, symbol Device:R
Connections:
- net GND: now also D?.1 (K), D?.1 (K), D?.1 (K), D?.1 (K), D?.1 (K), D?.1 (K), D?.1 (K), D?.1 (K), D?.1 (K), D?.1 (K), D?.1 (K)
- net Heater1: now also U6.2 (OUT2); no longer U6.6 (OUT1D)
- net Heater10: now also U6.25 (A11)
- net Heater11: now also U6.24 (A10)
- net Heater12: now also U6.23 (A9)
- net Heater2: now also U6.6 (OUT1D); no longer U6.9 (OUT1C)
- net Heater3: now also U6.9 (OUT1C); no longer U6.32 (OUT1B)
- net Heater4: now also U6.32 (OUT1B)
- net Heater5: now also U6.12 (MISO)
- net Heater6: now also U6.11 (MOSI)
- net Heater7: now also U6.38 (A14)
- net Heater8: now also U6.27 (A13)
- net Heater9: now also U6.26 (A12)
- net at U6.0 (RX1): now also R?.2
- net at U6.1 (TX1): now also R?.2
- net at U6.28 (RX7): now also R?.2
- net at U6.29 (TX7): now also R?.2
- net at U6.3 (LRCLK2): now also R?.2
- net at U6.30 (CRX3): now also R?.2
- net at U6.31 (CTX3): now also R?.2
- net at U6.34 (RX8): now also R?.2
- net at U6.35 (TX8): now also R?.2
- net at U6.7 (RX2): now also R?.2
- net at U6.8 (TX2): now also R?.2
- new net: D?.2 (A), R?.1 (x11)
- no-connect marks 40 -> 23

Commit message: Fixed schematic
Parts:
- removed C3: 22uF 50V, Capacitor_SMD:C_0603_1608Metric_Pad1.08x0.95mm_HandSolder, symbol Device:C_Polarized_US
- removed Conn? (x22): Molex_SL_02, symbol MRDT_Connectors:Molex_SL_02
- removed D? (x11): LED(B), LED_SMD:LED_0603_1608Metric_Pad1.05x0.95mm_HandSolder, symbol Device:LED
- removed F? (x12): 5, symbol Device:Fuse
- removed Q? (x11): IRF7606PBF, Package_SO:MSOP-8_3x3mm_P0.65mm, symbol Transistor_FET:IRF7606PBF
- removed Q? (x11): BSS138, Package_TO_SOT_SMD:SOT-23, symbol Transistor_FET:BSS138
- removed R? (x11): 1k, symbol Device:R
- removed R? (x22): 10k, symbol Device:R
- added Conn10, Conn11, Conn12, Conn13, Conn14, Conn15, Conn16, Conn17, Conn18, Conn19, Conn2, Conn20, Conn21, Conn22, Conn23, Conn24, Conn25, Conn3, Conn6, Conn7, Conn8, Conn9: Molex_SL_02, MRDT_Connectors:MOLEX_SL_02_Vertical, symbol MRDT_Connectors:Molex_SL_02
- added Conn26, Conn27, Conn28, Conn29, Conn30, Conn31, Conn32, Conn33, Conn34, Conn35, Conn36, Conn37: Molex_SL_03, MRDT_Connectors:MOLEX_SL_03_Vertical, symbol MRDT_Connectors:Molex_SL_03
- added D10, D11, D12, D13, D14, D15, D2, D6, D7, D8, D9: LED(B), LED_SMD:LED_0603_1608Metric_Pad1.05x0.95mm_HandSolder, symbol Device:LED
- added Q1, Q13, Q14, Q15, Q19, Q20, Q21, Q3, Q7, Q8, Q9: BSS138, Package_TO_SOT_SMD:SOT-23, symbol Transistor_FET:BSS138
- added Q10, Q11, Q12, Q16, Q17, Q18, Q22, Q23, Q24, Q4, Q6: IRF7606PBF, Package_SO:MSOP-8_3x3mm_P0.65mm, symbol Transistor_FET:IRF7606PBF
- added R1, R13, R14, R15, R16, R17, R18, R2, R22, R23, R24, R25, R26, R27, R31, R32, R33, R34, R35, R36, R7, R9: 10k, Resistor_SMD:R_0603_1608Metric_Pad0.98x0.95mm_HandSolder, symbol Device:R
- added R10, R12, R19, R20, R21, R28, R29, R30, R37, R38, R39: 1k, Resistor_SMD:R_0603_1608Metric_Pad0.98x0.95mm_HandSolder, symbol Device:R
- C7: value .1uF -> 10uF
- Conn4, Conn5: renamed from Conn?; footprint (none) -> MRDT_Connectors:MOLEX_SL_02_Vertical
- R11, R4, R40, R41, R42, R43, R44, R45, R46, R47, R48, R49, R5, R50: renamed from R?; footprint (none) -> Resistor_SMD:R_0603_1608Metric_Pad0.98x0.95mm_HandSolder
- gave numbers to parts that had none: 14
Connections:
- net +12V: now also C7.1, Q10.5 (D), Q10.6 (D), Q10.7 (D), Q10.8 (D), Q11.5 (D), Q11.6 (D), Q11.7 (D), Q11.8 (D), Q12.5 (D), Q12.6 (D), Q12.7 (D), Q12.8 (D), Q16.5 (D), Q16.6 (D), Q16.7 (D), Q16.8 (D), Q17.5 (D), Q17.6 (D), Q17.7 (D), Q17.8 (D), Q18.5 (D), Q18.6 (D), Q18.7 (D), Q18.8 (D), Q22.5 (D), Q22.6 (D), Q22.7 (D), Q22.8 (D), Q23.5 (D), Q23.6 (D), Q23.7 (D), Q23.8 (D), Q24.5 (D), Q24.6 (D), Q24.7 (D), Q24.8 (D), Q4.5 (D), Q4.6 (D), Q4.7 (D), Q4.8 (D), Q6.5 (D), Q6.6 (D), Q6.7 (D), Q6.8 (D), R1.1, R13.1, R15.1, R17.1, R22.1, R24.1, R26.1, R31.1, R33.1, R35.1, R7.1
- net +3V3: now also Conn26.1, Conn27.1, Conn28.1, Conn29.1, Conn30.1, Conn31.1, Conn32.1, Conn33.1, Conn34.1, Conn35.1, Conn36.1, Conn37.1; no longer C7.1
- net GND: now also Conn10.2, Conn11.2, Conn12.2, Conn13.2, Conn14.2, Conn15.2, Conn16.2, Conn17.2, Conn18.2, Conn19.2, Conn2.2, Conn20.2, Conn21.2, Conn22.2, Conn23.2, Conn24.2, Conn25.2, Conn26.3, Conn27.3, Conn28.3, Conn29.3, Conn3.2, Conn30.3, Conn31.3, Conn32.3, Conn33.3, Conn34.3, Conn35.3, Conn36.3, Conn37.3, Conn6.2, Conn7.2, Conn8.2, Conn9.2, D10.1 (K), D11.1 (K), D12.1 (K), D13.1 (K), D14.1 (K), D15.1 (K), D2.1 (K), D6.1 (K), D7.1 (K), D8.1 (K), D9.1 (K), Q1.2 (S), Q13.2 (S), Q14.2 (S), Q15.2 (S), Q19.2 (S), Q20.2 (S), Q21.2 (S), Q3.2 (S), Q7.2 (S), Q8.2 (S), Q9.2 (S)
- net Heater10: now also Q7.1 (G)
- net Heater11: now also Q13.1 (G)
- net Heater12: now also Q19.1 (G)
- net Heater2: now also Q8.1 (G)
- net Heater3: now also Q14.1 (G)
- net Heater4: now also Q20.1 (G)
- net Heater5: now also Q3.1 (G)
- net Heater6: now also Q9.1 (G)
- net Heater7: now also Q15.1 (G)
- net Heater8: now also Q21.1 (G)
- net Heater9: now also Q1.1 (G)
- net Temp1: now also Conn26.2; no longer Conn4.1, Conn5.1, Q5.1 (S), Q5.2 (S), Q5.3 (S), R11.1
- net Temp10: now also Conn36.2
- net Temp11: now also Conn31.2
- net Temp12: now also Conn37.2
- net Temp2: now also Conn32.2
- net Temp3: now also Conn27.2
- net Temp4: now also Conn33.2
- net Temp5: now also Conn28.2
- net Temp6: now also Conn34.2
- net Temp7: now also Conn29.2
- net Temp8: now also Conn35.2
- net Temp9: now also Conn30.2
- net at D3.2 (A): now also R11.1; no longer R11.2
- new net: Q24.4 (G), R35.2, R36.1
- new net: Q21.3 (D), R36.2
- new net: Q3.3 (D), R9.2
- new net: Q16.4 (G), R22.2, R23.1
- new net: Q13.3 (D), R23.2
- new net: Q9.3 (D), R18.2
- new net: Q12.4 (G), R17.2, R18.1
- new net: Conn22.1, Conn23.1, Q23.1 (S), Q23.2 (S), Q23.3 (S), R38.2
- new net: D7.2 (A), R19.1
- new net: Conn8.1, Conn9.1, Q10.1 (S), Q10.2 (S), Q10.3 (S), R19.2
- new net: Q14.3 (D), R25.2
- new net: D10.2 (A), R28.1
- new net: Conn14.1, Conn15.1, Q16.1 (S), Q16.2 (S), Q16.3 (S), R28.2
- new net: D14.2 (A), R38.1
- new net: Q8.3 (D), R16.2
- new net: Q10.4 (G), R13.2, R14.1
- new net: Q4.4 (G), R1.2, R2.1
- new net: Q1.3 (D), R2.2
- new net: D9.2 (A), R21.1
- new net: Conn12.1, Conn13.1, Q12.1 (S), Q12.2 (S), Q12.3 (S), R21.2
- new net: D11.2 (A), R29.1
- new net: Conn4.1, Conn5.1, Q5.1 (S), Q5.2 (S), Q5.3 (S), R11.2
- new net: Conn16.1, Conn17.1, Q17.1 (S), Q17.2 (S), Q17.3 (S), R29.2
- new net: Q17.4 (G), R24.2, R25.1
- new net: D6.2 (A), R12.1
- new net: Conn6.1, Conn7.1, Q6.1 (S), Q6.2 (S), Q6.3 (S), R12.2
- new net: D13.2 (A), R37.1
- new net: Conn20.1, Conn21.1, Q22.1 (S), Q22.2 (S), Q22.3 (S), R37.2
- new net: Q23.4 (G), R33.2, R34.1
- new net: Q20.3 (D), R34.2
- new net: Q18.4 (G), R26.2, R27.1
- new net: Q15.3 (D), R27.2
- new net: Q6.4 (G), R7.2, R9.1
- new net: Q7.3 (D), R14.2
- new net: Q22.4 (G), R31.2, R32.1
- new net: Conn10.1, Conn11.1, Q11.1 (S), Q11.2 (S), Q11.3 (S), R20.2
- new net: D2.2 (A), R10.1
- new net: Conn2.1, Conn3.1, Q4.1 (S), Q4.2 (S), Q4.3 (S), R10.2
- new net: Q11.4 (G), R15.2, R16.1
- new net: D12.2 (A), R30.1
- new net: Conn18.1, Conn19.1, Q18.1 (S), Q18.2 (S), Q18.3 (S), R30.2
- new net: Conn24.1, Conn25.1, Q24.1 (S), Q24.2 (S), Q24.3 (S), R39.2
- new net: D8.2 (A), R20.1
- new net: D15.2 (A), R39.1
- new net: Q19.3 (D), R32.2
Other:
- note added: "Temp Sensors"
- note added: "smirk"
- moved on the sheet: C7, Conn4, Conn5, D16, D17, D18, D19, D20, D21, D22, D23, D24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

Commit message: Placed heater block connectors
Connections:
- net +12V: now also Conn1.2 (V+Log); no longer Conn1.3 (V+Act)
- net TX+: now reaches J1.1, J2.1
- net TX-: now reaches J1.3, J2.2
- net RX-: now reaches J1.6, J2.5
- net RX+: now reaches J1.4, J2.6
Changed lines of the file:
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@@
     (effects (font (size 25 25) (thickness 1) bold italic) (justify left bottom))
   )
+  (label "TX+" (at 255.27 153.67 0)
+    (effects (font (size 1.27 1.27)) (justify left bottom))
+  )
+  (label "RX-" (at 255.905 143.51 0)
+    (effects (font (size 1.27 1.27)) (justify left bottom))
+  )
+  (label "TX-" (at 255.905 151.13 0)
+    (effects (font (size 1.27 1.27)) (justify left bottom))
+  )
+  (label "RX+" (at 257.175 138.43 0)
+    (effects (font (size 1.27 1.27)) (justify left bottom))
+  )
   (global_label "Heater10" (shape output) (at 255.27 107.95 0) (fields_autoplaced)
     (effects (font (size 1.27 1.27)) (justify left))
@@
   (symbol (lib_id "power:+12V") (at 33.02 149.86 0) (unit 1)
     (in_bom yes) (on_board yes) (fields_autoplaced)
-    (property "Reference" "#PWR?" (id 0) (at 33.02 153.67 0)
+    (property "Reference" "#PWR0109" (id 0) (at 33.02 153.67 0)
       (effects (font (size 1.27 1.27)) hide)
     )
@@
   (symbol (lib_id "power:+12V") (at 113.03 149.86 0) (unit 1)
     (in_bom yes) (on_board yes) (fields_autoplaced)
-    (property "Reference" "#PWR?" (id 0) (at 113.03 153.67 0)
+    (property "Reference" "#PWR0117" (id 0) (at 113.03 153.67 0)
       (effects (font (size 1.27 1.27)) hide)
     )
@@
   (symbol (lib_id "power:+12V") (at 73.66 60.325 0) (unit 1)
     (in_bom yes) (on_board yes) (fields_autoplaced)
-    (property "Reference" "#PWR?" (id 0) (at 73.66 64.135 0)
+    (property "Reference" "#PWR0116" (id 0) (at 73.66 64.135 0)
       (effects (font (size 1.27 1.27)) hide)
     )
@@
   (symbol (lib_id "power:+12V") (at 153.67 60.325 0) (unit 1)
     (in_bom yes) (on_board yes) (fields_autoplaced)
-    (property "Reference" "#PWR?" (id 0) (at 153.67 64.135 0)
+    (property "Reference" "#PWR0112" (id 0) (at 153.67 64.135 0)
       (effects (font (size 1.27 1.27)) hide)
     )
@@
   (symbol (lib_id "power:+12V") (at 73.66 104.775 0) (unit 1)
     (in_bom yes) (on_board yes) (fields_autoplaced)
-    (property "Reference" "#PWR?" (id 0) (at 73.66 108.585 0)
+    (property "Reference" "#PWR0107" (id 0) (at 73.66 108.585 0)
       (effects (font (size 1.27 1.27)) hide)
     )
@@
   (symbol (lib_id "power:+12V") (at 73.025 149.86 0) (unit 1)
     (in_bom yes) (on_board yes) (fields_autoplaced)
-    (property "Reference" "#PWR?" (id 0) (at 73.025 153.67 0)
+    (property "Reference" "#PWR0108" (id 0) (at 73.025 153.67 0)
       (effects (font (size 1.27 1.27)) hide)
     )
@@
   (symbol (lib_id "power:+12V") (at 153.67 104.775 0) (unit 1)
     (in_bom yes) (on_board yes) (fields_autoplaced)
-    (property "Reference" "#PWR?" (id 0) (at 153.67 108.585 0)
+    (property "Reference" "#PWR0115" (id 0) (at 153.67 108.585 0)
       (effects (font (size 1.27 1.27)) hide)
     )
@@
     (pin "2")
   )
-  (symbol (lib_id "MRDT_Connectors:AndersonPP") (at 16.51 41.91 0) (unit 3)
+  (symbol (lib_id "MRDT_Connectors:AndersonPP") (at 16.51 41.91 0) (unit 2)
     (in_bom yes) (on_board yes) (fields_autoplaced)
     (property "Reference" "Conn1" (id 0) (at 19.05 31.75 0)
@@
   (symbol (lib_id "power:+12V") (at 153.035 149.86 0) (unit 1)
     (in_bom yes) (on_board yes) (fields_autoplaced)
-    (property "Reference" "#PWR?" (id 0) (at 153.035 153.67 0)
+    (property "Reference" "#PWR0103" (id 0) (at 153.035 153.67 0)
       (effects (font (size 1.27 1.27)) hide)
     )
@@
   (symbol (lib_id "power:+12V") (at 113.665 60.325 0) (unit 1)
     (in_bom yes) (on_board yes) (fields_autoplaced)
-    (property "Reference" "#PWR?" (id 0) (at 113.665 64.135 0)
+    (property "Reference" "#PWR0113" (id 0) (at 113.665 64.135 0)
       (effects (font (size 1.27 1.27)) hide)
     )
@@
   (symbol (lib_id "power:+12V") (at 113.665 104.775 0) (unit 1)
     (in_bom yes) (on_board yes) (fields_autoplaced)
-    (property "Reference" "#PWR?" (id 0) (at 113.665 108.585 0)
+    (property "Reference" "#PWR0114" (id 0) (at 113.665 108.585 0)
       (effects (font (size 1.27 1.27)) hide)
     )
@@
   (symbol (lib_id "power:+12V") (at 33.655 104.775 0) (unit 1)
     (in_bom yes) (on_board yes) (fields_autoplaced)
-    (property "Reference" "#PWR?" (id 0) (at 33.655 108.585 0)
+    (property "Reference" "#PWR0105" (id 0) (at 33.655 108.585 0)
       (effects (font (size 1.27 1.27)) hide)
     )
@@
       (reference "#PWR0102") (unit 1) (value "+12V") (footprint "")
     )
+    (path "/ad175320-019b-40e4-8a4c-fbb6a8b65e61"
+      (reference "#PWR0103") (unit 1) (value "+12V") (footprint "")
+    )
     (path "/75394c0e-8deb-4c1b-96d9-90a95f192003"
       (reference "#PWR0104") (unit 1) (value "GND") (footprint "")
     )
+    (path "/f1a9f7fa-2d61-4019-93e7-8dcb426dbf7a"
+      (reference "#PWR0105") (unit 1) (value "+12V") (footprint "")
+    )
     (path "/f831749c-8854-41e2-96ff-34e6e71e9ae8"
       (reference "#PWR0106") (unit 1) (value "GND") (footprint "")
     )
+    (path "/482e7a94-191c-494d-a365-ac8498130284"
+      (reference "#PWR0107") (unit 1) (value "+12V") (footprint "")
+    )
+    (path "/49d0de4b-12b4-45b2-9afb-09da4df9e058"
+      (reference "#PWR0108") (unit 1) (value "+12V") (footprint "")
+    )
+    (path "/0910aa4b-6918-402c-8e96-af5e1bb9651e"
+      (reference "#PWR0109") (unit 1) (value "+12V") (footprint "")
+    )
     (path "/63c3fe76-6fde-4d6c-afb2-01ec61b588d5"
       (reference "#PWR0110") (unit 1) (value "GND") (footprint "")
@@
       (reference "#PWR0111") (unit 1) (value "+12V") (footprint "")
     )
+    (path "/360b9b3f-6828-4e31-9191-f3b49b69aab6"
+      (reference "#PWR0112") (unit 1) (value "+12V") (footprint "")
+    )
+    (path "/c85aacbe-9a8a-4ec0-b24f-c44ed8a6f0da"
+      (reference "#PWR0113") (unit 1) (value "+12V") (footprint "")
+    )
+    (path "/ce68fc82-a51b-4262-9255-91bce48a0916"
+      (reference "#PWR0114") (unit 1) (value "+12V") (footprint "")
+    )
+    (path "/87636ed8-1aaa-4d94-ba9a-95ab61c58e97"
+      (reference "#PWR0115") (unit 1) (value "+12V") (footprint "")
+    )
+    (path "/34bc49e3-a0e3-4577-b5e4-692e7678ee68"
+      (reference "#PWR0116") (unit 1) (value "+12V") (footprint "")
+    )
+    (path "/20f7674a-b56a-40d4-a310-f134ab67b5ac"
+      (reference "#PWR0117") (unit 1) (value "+12V") (footprint "")
+    )
     (path "/7bcab7ed-fe56-4d9a-87ca-c720f26731de"
       (reference "#PWR0122") (unit 1) (value "GND") (footprint "")
@@
       (reference "#PWR0128") (unit 1) (value "+3V3") (footprint "")
     )
-    (path "/0910aa4b-6918-402c-8e96-af5e1bb9651e"
-      (reference "#PWR?") (unit 1) (value "+12V") (footprint "")
-    )
-    (path "/20f7674a-b56a-40d4-a310-f134ab67b5ac"
-      (reference "#PWR?") (unit 1) (value "+12V") (footprint "")
-    )
-    (path "/34bc49e3-a0e3-4577-b5e4-692e7678ee68"
-      (reference "#PWR?") (unit 1) (value "+12V") (footprint "")
-    )
-    (path "/360b9b3f-6828-4e31-9191-f3b49b69aab6"
-      (reference "#PWR?") (unit 1) (value "+12V") (footprint "")
-    )
-    (path "/482e7a94-191c-494d-a365-ac8498130284"
-      (reference "#PWR?") (unit 1) (value "+12V") (footprint "")
-    )
-    (path "/49d0de4b-12b4-45b2-9afb-09da4df9e058"
-      (reference "#PWR?") (unit 1) (value "+12V") (footprint "")
-    )
-    (path "/87636ed8-1aaa-4d94-ba9a-95ab61c58e97"
-      (reference "#PWR?") (unit 1) (value "+12V") (footprint "")
-    )
-    (path "/ad175320-019b-40e4-8a4c-fbb6a8b65e61"
-      (reference "#PWR?") (unit 1) (value "+12V") (footprint "")
-    )
-    (path "/c85aacbe-9a8a-4ec0-b24f-c44ed8a6f0da"
-      (reference "#PWR?") (unit 1) (value "+12V") (footprint "")
-    )
-    (path "/ce68fc82-a51b-4262-9255-91bce48a0916"
-      (reference "#PWR?") (unit 1) (value "+12V") (footprint "")
-    )
-    (path "/f1a9f7fa-2d61-4019-93e7-8dcb426dbf7a"
-      (reference "#PWR?") (unit 1) (value "+12V") (footprint "")
-    )
     (path "/62260b31-0a19-47a4-af9d-4d902abd11b6"
       (reference "C6") (unit 1) (value "10uF") (footprint "Capacitor_SMD:C_0603_1608Metric_Pad1.08x0.95mm_HandSolder")
@@
     )
     (path "/9f08d595-5234-481a-8f49-8981e5969103"
-      (reference "Conn1") (unit 3) (value "AndersonPP") (footprint "MRDT_Connectors:Anderson_2_Horizontal_Side_by_Side")
+      (reference "Conn1") (unit 2) (value "AndersonPP") (footprint "MRDT_Connectors:Anderson_2_Horizontal_Side_by_Side")
     )
     (path "/8ed15565-e6e8-46cc-9fed-3b113c5c5619"

Commit message: Worked on connector placements
Connections:
- net +12V: now also Q5.5 (D), Q5.6 (D), Q5.7 (D), Q5.8 (D), R4.1
Changed lines of the file:
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@@
   (junction (at 165.735 88.9) (diameter 0) (color 0 0 0 0)
   )
+  (junction (at 33.655 63.5) (diameter 0) (color 0 0 0 0)
+  )
   (junction (at 45.72 77.47) (diameter 0) (color 0 0 0 0)
   )
@@
     (stroke (width 0) (type default) (color 0 0 0 0))
   )
+  (wire (pts (xy 33.655 60.325) (xy 33.655 63.5))
+    (stroke (width 0) (type default) (color 0 0 0 0))
+  )
   (wire (pts (xy 22.225 116.332) (xy 22.225 116.84))
     (stroke (width 0) (type default) (color 0 0 0 0))
@@
     (pin "3")
   )
+  (symbol (lib_id "power:+12V") (at 33.655 60.325 0) (unit 1)
+    (in_bom yes) (on_board yes) (fields_autoplaced)
+    (property "Reference" "#PWR?" (id 0) (at 33.655 64.135 0)
+      (effects (font (size 1.27 1.27)) hide)
+    )
+    (property "Value" "+12V" (id 1) (at 33.655 56.7492 0))
+    (property "Footprint" "" (id 2) (at 33.655 60.325 0)
+      (effects (font (size 1.27 1.27)) hide)
+    )
+    (property "Datasheet" "" (id 3) (at 33.655 60.325 0)
+      (effects (font (size 1.27 1.27)) hide)
+    )
+    (pin "1")
+  )
   (symbol (lib_id "Device:R") (at 142.24 67.31 0) (unit 1)
     (in_bom yes) (on_board yes)
@@
       (reference "#PWR0128") (unit 1) (value "+3V3") (footprint "")
     )
+    (path "/865efa5d-ece8-49ad-8a45-c661d4660d3d"
+      (reference "#PWR?") (unit 1) (value "+12V") (footprint "")
+    )
     (path "/62260b31-0a19-47a4-af9d-4d902abd11b6"
