File: hardware/Hardware_Rev1.kicad_sch (KiCad schematic)
At the start: 160 parts, among them J1 RJ45_LED_Shielded, J2 6P6C, Q1 BSS138, Q10 AO3401A, Q11 AO3401A, Q12 AO3401A, Q13 BSS138, Q14 BSS138, Q15 BSS138, Q16 AO3401A, Q17 AO3401A, Q18 AO3401A, Q19 BSS138, Q2 BSS138, Q20 BSS138, Q21 BSS138, Q22 AO3401A, Q23 AO3401A, Q24 AO3401A, Q3 BSS138, Q4 AO3401A, Q5 AO3401A, Q6 AO3401A, Q7 BSS138, Q8 BSS138, Q9 BSS138, U1 OKI, U2 Teensy4.1_DEV-16771

Commit message: Made layout review changes
Parts:
- Conn1: footprint MRDT_Connectors:Anderson_2_Horizontal_Side_by_Side -> MRDT_Connectors:Square_Anderson_2_H_Side_By_Side
Connections:
- net at U2.0 (RX1): now also R48.2; no longer R47.2
- net at U2.1 (TX1): now also R47.2; no longer R48.2
Other:
- moved on the sheet: D23, D24, R47, R48
Changed lines of the file:
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@@
     (stroke (width 0) (type default) (color 0 0 0 0))
   )
-  (wire (pts (xy 200.66 52.07) (xy 202.565 52.07))
+  (wire (pts (xy 200.66 54.61) (xy 202.565 54.61))
     (stroke (width 0) (type default) (color 0 0 0 0))
   )
@@
     (stroke (width 0) (type default) (color 0 0 0 0))
   )
-  (wire (pts (xy 200.66 54.61) (xy 202.565 54.61))
+  (wire (pts (xy 200.66 52.07) (xy 202.565 52.07))
     (stroke (width 0) (type default) (color 0 0 0 0))
   )
@@
   (symbol (lib_id "power:GND") (at 191.77 60.96 0) (mirror y) (unit 1)
     (in_bom yes) (on_board yes) (fields_autoplaced)
-    (property "Reference" "#PWR?" (id 0) (at 191.77 67.31 0)
+    (property "Reference" "#PWR0106" (id 0) (at 191.77 67.31 0)
       (effects (font (size 1.27 1.27)) hide)
     )
@@
       (effects (font (size 1.524 1.524)))
     )
-    (property "Footprint" "MRDT_Connectors:Anderson_2_Horizontal_Side_by_Side" (id 2) (at 12.7 41.91 0)
+    (property "Footprint" "MRDT_Connectors:Square_Anderson_2_H_Side_By_Side" (id 2) (at 12.7 41.91 0)
       (effects (font (size 1.524 1.524)) hide)
     )
@@
     (pin "2")
   )
-  (symbol (lib_id "Device:LED") (at 196.85 52.07 0) (unit 1)
+  (symbol (lib_id "Device:LED") (at 196.85 54.61 0) (unit 1)
     (in_bom yes) (on_board yes)
-    (property "Reference" "D23" (id 0) (at 199.136 52.832 0)
+    (property "Reference" "D23" (id 0) (at 199.136 55.372 0)
       (effects (font (size 0.889 0.889)))
     )
-    (property "Value" "LED(R)" (id 1) (at 200.406 51.308 0)
+    (property "Value" "LED(R)" (id 1) (at 200.406 53.848 0)
       (effects (font (size 0.889 0.889)))
     )
-    (property "Footprint" "LED_SMD:LED_0603_1608Metric_Pad1.05x0.95mm_HandSolder" (id 2) (at 196.85 52.07 0)
+    (property "Footprint" "LED_SMD:LED_0603_1608Metric_Pad1.05x0.95mm_HandSolder" (id 2) (at 196.85 54.61 0)
       (effects (font (size 1.27 1.27)) hide)
     )
-    (property "Datasheet" "~" (id 3) (at 196.85 52.07 0)
+    (property "Datasheet" "~" (id 3) (at 196.85 54.61 0)
       (effects (font (size 1.27 1.27)) hide)
     )
@@
     (pin "2")
   )
-  (symbol (lib_id "Device:R") (at 206.375 54.61 90) (unit 1)
+  (symbol (lib_id "Device:R") (at 206.375 52.07 90) (unit 1)
     (in_bom yes) (on_board yes)
-    (property "Reference" "R48" (id 0) (at 210.82 53.975 90))
-    (property "Value" "120" (id 1) (at 206.375 54.61 90))
-    (property "Footprint" "Resistor_SMD:R_0603_1608Metric_Pad0.98x0.95mm_HandSolder" (id 2) (at 206.375 56.388 90)
+    (property "Reference" "R48" (id 0) (at 210.82 51.435 90))
+    (property "Value" "120" (id 1) (at 206.375 52.07 90))
+    (property "Footprint" "Resistor_SMD:R_0603_1608Metric_Pad0.98x0.95mm_HandSolder" (id 2) (at 206.375 53.848 90)
       (effects (font (size 1.27 1.27)) hide)
     )
-    (property "Datasheet" "~" (id 3) (at 206.375 54.61 0)
+    (property "Datasheet" "~" (id 3) (at 206.375 52.07 0)
       (effects (font (size 1.27 1.27)) hide)
     )
@@
       (effects (font (size 1.524 1.524)))
     )
-    (property "Footprint" "MRDT_Connectors:Anderson_2_Horizontal_Side_by_Side" (id 2) (at 12.7 55.88 0)
+    (property "Footprint" "MRDT_Connectors:Square_Anderson_2_H_Side_By_Side" (id 2) (at 12.7 55.88 0)
       (effects (font (size 1.524 1.524)) hide)
     )
@@
     (pin "2")
   )
-  (symbol (lib_id "Device:LED") (at 196.85 54.61 0) (unit 1)
+  (symbol (lib_id "Device:LED") (at 196.85 52.07 0) (unit 1)
     (in_bom yes) (on_board yes)
-    (property "Reference" "D24" (id 0) (at 199.136 55.372 0)
+    (property "Reference" "D24" (id 0) (at 199.136 52.832 0)
       (effects (font (size 0.889 0.889)))
     )
-    (property "Value" "LED(R)" (id 1) (at 200.406 53.848 0)
+    (property "Value" "LED(R)" (id 1) (at 200.406 51.308 0)
       (effects (font (size 0.889 0.889)))
     )
-    (property "Footprint" "LED_SMD:LED_0603_1608Metric_Pad1.05x0.95mm_HandSolder" (id 2) (at 196.85 54.61 0)
+    (property "Footprint" "LED_SMD:LED_0603_1608Metric_Pad1.05x0.95mm_HandSolder" (id 2) (at 196.85 52.07 0)
       (effects (font (size 1.27 1.27)) hide)
     )
-    (property "Datasheet" "~" (id 3) (at 196.85 54.61 0)
+    (property "Datasheet" "~" (id 3) (at 196.85 52.07 0)
       (effects (font (size 1.27 1.27)) hide)
     )
@@
     (pin "2")
   )
-  (symbol (lib_id "Device:R") (at 206.375 52.07 90) (unit 1)
+  (symbol (lib_id "Device:R") (at 206.375 54.61 90) (unit 1)
     (in_bom yes) (on_board yes)
-    (property "Reference" "R47" (id 0) (at 210.82 51.435 90))
-    (property "Value" "120" (id 1) (at 206.375 52.07 90))
-    (property "Footprint" "Resistor_SMD:R_0603_1608Metric_Pad0.98x0.95mm_HandSolder" (id 2) (at 206.375 53.848 90)
+    (property "Reference" "R47" (id 0) (at 210.82 53.975 90))
+    (property "Value" "120" (id 1) (at 206.375 54.61 90))
+    (property "Footprint" "Resistor_SMD:R_0603_1608Metric_Pad0.98x0.95mm_HandSolder" (id 2) (at 206.375 56.388 90)
       (effects (font (size 1.27 1.27)) hide)
     )
-    (property "Datasheet" "~" (id 3) (at 206.375 52.07 0)
+    (property "Datasheet" "~" (id 3) (at 206.375 54.61 0)
       (effects (font (size 1.27 1.27)) hide)
     )
@@
     )
     (path "/1a3a5818-0fcd-4d75-8a88-681dbca64019"
-      (reference "#PWR?") (unit 1) (value "GND") (footprint "")
+      (reference "#PWR0106") (unit 1) (value "GND") (footprint "")
     )
     (path "/14a93ed5-04ed-45a3-bcf0-d259f23ab9ae"
@@
     )
     (path "/51fe58c1-957c-49ab-ba18-9946891c75e6"
-      (reference "Conn1") (unit 1) (value "AndersonPP") (footprint "MRDT_Connectors:Anderson_2_Horizontal_Side_by_Side")
+      (reference "Conn1") (unit 1) (value "AndersonPP") (footprint "MRDT_Connectors:Square_Anderson_2_H_Side_By_Side")
     )
     (path "/9f08d595-5234-481a-8f49-8981e5969103"
-      (reference "Conn1") (unit 2) (value "AndersonPP") (footprint "MRDT_Connectors:Anderson_2_Horizontal_Side_by_Side")
+      (reference "Conn1") (unit 2) (value "AndersonPP") (footprint "MRDT_Connectors:Square_Anderson_2_H_Side_By_Side")
     )
     (path "/8ed15565-e6e8-46cc-9fed-3b113c5c5619"

Commit message: Changed teensy footprint
Parts:
- U2: footprint MRDT_Shields:Teensy_4_1_Vertical -> MRDT_Shields:Teensy_4_1_Bare
Changed lines of the file:
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@@
     (property "Reference" "U2" (id 0) (at 234.315 18.415 0))
     (property "Value" "Teensy4.1_DEV-16771" (id 1) (at 234.95 20.32 0))
-    (property "Footprint" "MRDT_Shields:Teensy_4_1_Vertical" (id 2) (at 287.02 80.01 0)
+    (property "Footprint" "MRDT_Shields:Teensy_4_1_Bare" (id 2) (at 287.02 80.01 0)
       (effects (font (size 1.27 1.27)) (justify left bottom) hide)
     )
@@
     )
     (path "/165afba2-0703-4f13-aa69-df8fca3cdcf1"
-      (reference "U2") (unit 1) (value "Teensy4.1_DEV-16771") (footprint "MRDT_Shields:Teensy_4_1_Vertical")
+      (reference "U2") (unit 1) (value "Teensy4.1_DEV-16771") (footprint "MRDT_Shields:Teensy_4_1_Bare")
     )
     (path "/8053e13e-7718-49bc-b6d0-eac399e3fb77"
