File: hardware/Hardware_Rev1.kicad_sch (KiCad schematic)
At the start: 150 parts, among them J1 RJ45_LED_Shielded, Q1 BSS138, Q10 Q_PMOS_GSD, Q11 Q_PMOS_GSD, Q12 Q_PMOS_GSD, Q13 BSS138, Q14 BSS138, Q15 BSS138, Q16 Q_PMOS_GSD, Q17 Q_PMOS_GSD, Q18 Q_PMOS_GSD, Q19 BSS138, Q2 BSS138, Q20 BSS138, Q21 BSS138, Q22 Q_PMOS_GSD, Q23 Q_PMOS_GSD, Q24 Q_PMOS_GSD, Q3 BSS138, Q4 Q_PMOS_GSD, Q5 Q_PMOS_GSD, Q6 Q_PMOS_GSD, Q7 BSS138, Q8 BSS138, Q9 BSS138, U1 OKI, U2 Teensy4.1_DEV-16771

Commit message: Fixed pfet connections
Connections:
- net +12V: now also Q10.2 (S), Q11.2 (S), Q12.2 (S), Q16.2 (S), Q17.2 (S), Q18.2 (S), Q22.2 (S), Q23.2 (S), Q24.2 (S), Q4.2 (S), Q5.2 (S), Q6.2 (S); no longer Q10.3 (D), Q11.3 (D), Q12.3 (D), Q16.3 (D), Q17.3 (D), Q18.3 (D), Q22.3 (D), Q23.3 (D), Q24.3 (D), Q4.3 (D), Q5.3 (D), Q6.3 (D)
- net H1: now also Q5.3 (D); no longer Q5.2 (S)
- net H10: now also Q10.3 (D); no longer Q10.2 (S)
- net H11: now also Q17.3 (D); no longer Q17.2 (S)
- net H12: now also Q22.3 (D); no longer Q22.2 (S)
- net H2: now also Q11.3 (D); no longer Q11.2 (S)
- net H3: now also Q16.3 (D); no longer Q16.2 (S)
- net H4: now also Q23.3 (D); no longer Q23.2 (S)
- net H5: now also Q6.3 (D); no longer Q6.2 (S)
- net H6: now also Q12.3 (D); no longer Q12.2 (S)
- net H7: now also Q18.3 (D); no longer Q18.2 (S)
- net H8: now also Q24.3 (D); no longer Q24.2 (S)
- net H9: now also Q4.3 (D); no longer Q4.2 (S)
Changed lines of the file:
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@@
     (pin "1")
   )
-  (symbol (lib_id "Device:Q_PMOS_GSD") (at 110.49 71.755 0) (unit 1)
+  (symbol (lib_id "Device:Q_PMOS_GSD") (at 110.49 71.755 0) (mirror x) (unit 1)
     (in_bom yes) (on_board yes)
     (property "Reference" "Q16" (id 0) (at 115.57 71.755 0)
       (effects (font (size 1.27 1.27)) (justify left))
     )
-    (property "Value" "Q_PMOS_GSD" (id 1) (at 104.775 67.945 0)
+    (property "Value" "Q_PMOS_GSD" (id 1) (at 104.775 75.565 0)
       (effects (font (size 1.27 1.27)) (justify left))
     )
-    (property "Footprint" "Package_TO_SOT_SMD:SOT-23-3" (id 2) (at 115.57 69.215 0)
+    (property "Footprint" "Package_TO_SOT_SMD:SOT-23-3" (id 2) (at 115.57 74.295 0)
       (effects (font (size 1.27 1.27)) hide)
     )
@@
     (pin "1")
   )
-  (symbol (lib_id "Device:Q_PMOS_GSD") (at 31.115 116.205 0) (unit 1)
+  (symbol (lib_id "Device:Q_PMOS_GSD") (at 31.115 116.205 0) (mirror x) (unit 1)
     (in_bom yes) (on_board yes)
     (property "Reference" "Q6" (id 0) (at 36.195 116.205 0)
       (effects (font (size 1.27 1.27)) (justify left))
     )
-    (property "Value" "Q_PMOS_GSD" (id 1) (at 25.4 112.395 0)
+    (property "Value" "Q_PMOS_GSD" (id 1) (at 25.4 120.015 0)
       (effects (font (size 1.27 1.27)) (justify left))
     )
-    (property "Footprint" "Package_TO_SOT_SMD:SOT-23-3" (id 2) (at 36.195 113.665 0)
+    (property "Footprint" "Package_TO_SOT_SMD:SOT-23-3" (id 2) (at 36.195 118.745 0)
       (effects (font (size 1.27 1.27)) hide)
     )
@@
     (pin "2")
   )
-  (symbol (lib_id "Device:Q_PMOS_GSD") (at 30.48 161.29 0) (unit 1)
+  (symbol (lib_id "Device:Q_PMOS_GSD") (at 30.48 161.29 0) (mirror x) (unit 1)
     (in_bom yes) (on_board yes)
     (property "Reference" "Q4" (id 0) (at 35.56 161.29 0)
       (effects (font (size 1.27 1.27)) (justify left))
     )
-    (property "Value" "Q_PMOS_GSD" (id 1) (at 24.765 157.48 0)
+    (property "Value" "Q_PMOS_GSD" (id 1) (at 24.765 165.1 0)
       (effects (font (size 1.27 1.27)) (justify left))
     )
-    (property "Footprint" "Package_TO_SOT_SMD:SOT-23-3" (id 2) (at 35.56 158.75 0)
+    (property "Footprint" "Package_TO_SOT_SMD:SOT-23-3" (id 2) (at 35.56 163.83 0)
       (effects (font (size 1.27 1.27)) hide)
     )
@@
     (pin "2")
   )
-  (symbol (lib_id "Device:Q_PMOS_GSD") (at 71.12 161.29 0) (unit 1)
+  (symbol (lib_id "Device:Q_PMOS_GSD") (at 71.12 161.29 0) (mirror x) (unit 1)
     (in_bom yes) (on_board yes)
     (property "Reference" "Q10" (id 0) (at 76.2 161.29 0)
       (effects (font (size 1.27 1.27)) (justify left))
     )
-    (property "Value" "Q_PMOS_GSD" (id 1) (at 65.405 157.48 0)
+    (property "Value" "Q_PMOS_GSD" (id 1) (at 65.405 165.1 0)
       (effects (font (size 1.27 1.27)) (justify left))
     )
-    (property "Footprint" "Package_TO_SOT_SMD:SOT-23-3" (id 2) (at 76.2 158.75 0)
+    (property "Footprint" "Package_TO_SOT_SMD:SOT-23-3" (id 2) (at 76.2 163.83 0)
       (effects (font (size 1.27 1.27)) hide)
     )
@@
     (pin "1")
   )
-  (symbol (lib_id "Device:Q_PMOS_GSD") (at 110.49 161.29 0) (unit 1)
+  (symbol (lib_id "Device:Q_PMOS_GSD") (at 110.49 161.29 0) (mirror x) (unit 1)
     (in_bom yes) (on_board yes)
     (property "Reference" "Q17" (id 0) (at 115.57 161.29 0)
       (effects (font (size 1.27 1.27)) (justify left))
     )
-    (property "Value" "Q_PMOS_GSD" (id 1) (at 104.775 157.48 0)
+    (property "Value" "Q_PMOS_GSD" (id 1) (at 104.775 165.1 0)
       (effects (font (size 1.27 1.27)) (justify left))
     )
-    (property "Footprint" "Package_TO_SOT_SMD:SOT-23-3" (id 2) (at 115.57 158.75 0)
+    (property "Footprint" "Package_TO_SOT_SMD:SOT-23-3" (id 2) (at 115.57 163.83 0)
       (effects (font (size 1.27 1.27)) hide)
     )
@@
     (pin "1")
   )
-  (symbol (lib_id "Device:Q_PMOS_GSD") (at 151.13 116.205 0) (unit 1)
+  (symbol (lib_id "Device:Q_PMOS_GSD") (at 151.13 116.205 0) (mirror x) (unit 1)
     (in_bom yes) (on_board yes)
     (property "Reference" "Q24" (id 0) (at 156.21 116.205 0)
       (effects (font (size 1.27 1.27)) (justify left))
     )
-    (property "Value" "Q_PMOS_GSD" (id 1) (at 145.415 112.395 0)
+    (property "Value" "Q_PMOS_GSD" (id 1) (at 145.415 120.015 0)
       (effects (font (size 1.27 1.27)) (justify left))
     )
-    (property "Footprint" "Package_TO_SOT_SMD:SOT-23-3" (id 2) (at 156.21 113.665 0)
+    (property "Footprint" "Package_TO_SOT_SMD:SOT-23-3" (id 2) (at 156.21 118.745 0)
       (effects (font (size 1.27 1.27)) hide)
     )
@@
     (pin "3")
   )
-  (symbol (lib_id "Device:Q_PMOS_GSD") (at 31.115 71.755 0) (unit 1)
+  (symbol (lib_id "Device:Q_PMOS_GSD") (at 31.115 71.755 0) (mirror x) (unit 1)
     (in_bom yes) (on_board yes)
     (property "Reference" "Q5" (id 0) (at 36.195 71.755 0)
       (effects (font (size 1.27 1.27)) (justify left))
     )
-    (property "Value" "Q_PMOS_GSD" (id 1) (at 25.4 67.945 0)
+    (property "Value" "Q_PMOS_GSD" (id 1) (at 25.4 75.565 0)
       (effects (font (size 1.27 1.27)) (justify left))
     )
-    (property "Footprint" "Package_TO_SOT_SMD:SOT-23-3" (id 2) (at 36.195 69.215 0)
+    (property "Footprint" "Package_TO_SOT_SMD:SOT-23-3" (id 2) (at 36.195 74.295 0)
       (effects (font (size 1.27 1.27)) hide)
     )
@@
     (pin "2")
   )
-  (symbol (lib_id "Device:Q_PMOS_GSD") (at 71.12 116.205 0) (unit 1)
+  (symbol (lib_id "Device:Q_PMOS_GSD") (at 71.12 116.205 0) (mirror x) (unit 1)
     (in_bom yes) (on_board yes)
     (property "Reference" "Q12" (id 0) (at 76.2 116.205 0)
       (effects (font (size 1.27 1.27)) (justify left))
     )
-    (property "Value" "Q_PMOS_GSD" (id 1) (at 65.405 112.395 0)
+    (property "Value" "Q_PMOS_GSD" (id 1) (at 65.405 120.015 0)
       (effects (font (size 1.27 1.27)) (justify left))
     )
-    (property "Footprint" "Package_TO_SOT_SMD:SOT-23-3" (id 2) (at 76.2 113.665 0)
+    (property "Footprint" "Package_TO_SOT_SMD:SOT-23-3" (id 2) (at 76.2 118.745 0)
       (effects (font (size 1.27 1.27)) hide)
     )
@@
     (pin "2")
   )
-  (symbol (lib_id "Device:Q_PMOS_GSD") (at 151.13 161.29 0) (unit 1)
+  (symbol (lib_id "Device:Q_PMOS_GSD") (at 151.13 161.29 0) (mirror x) (unit 1)
     (in_bom yes) (on_board yes)
     (property "Reference" "Q22" (id 0) (at 156.21 161.29 0)
       (effects (font (size 1.27 1.27)) (justify left))
     )
-    (property "Value" "Q_PMOS_GSD" (id 1) (at 145.415 157.48 0)
+    (property "Value" "Q_PMOS_GSD" (id 1) (at 145.415 165.1 0)
       (effects (font (size 1.27 1.27)) (justify left))
     )
-    (property "Footprint" "Package_TO_SOT_SMD:SOT-23-3" (id 2) (at 156.21 158.75 0)
+    (property "Footprint" "Package_TO_SOT_SMD:SOT-23-3" (id 2) (at 156.21 163.83 0)
       (effects (font (size 1.27 1.27)) hide)
     )
@@
     (pin "3")
   )
-  (symbol (lib_id "Device:Q_PMOS_GSD") (at 151.13 71.755 0) (unit 1)
+  (symbol (lib_id "Device:Q_PMOS_GSD") (at 151.13 71.755 0) (mirror x) (unit 1)
     (in_bom yes) (on_board yes)
     (property "Reference" "Q23" (id 0) (at 156.21 71.755 0)
       (effects (font (size 1.27 1.27)) (justify left))
     )
-    (property "Value" "Q_PMOS_GSD" (id 1) (at 145.415 67.945 0)
+    (property "Value" "Q_PMOS_GSD" (id 1) (at 145.415 75.565 0)
       (effects (font (size 1.27 1.27)) (justify left))
     )
-    (property "Footprint" "Package_TO_SOT_SMD:SOT-23-3" (id 2) (at 156.21 69.215 0)
+    (property "Footprint" "Package_TO_SOT_SMD:SOT-23-3" (id 2) (at 156.21 74.295 0)
       (effects (font (size 1.27 1.27)) hide)
     )
@@
     (pin "1")
   )
-  (symbol (lib_id "Device:Q_PMOS_GSD") (at 71.12 71.755 0) (unit 1)
+  (symbol (lib_id "Device:Q_PMOS_GSD") (at 71.12 71.755 0) (mirror x) (unit 1)
     (in_bom yes) (on_board yes)
     (property "Reference" "Q11" (id 0) (at 76.2 71.755 0)
       (effects (font (size 1.27 1.27)) (justify left))
     )
-    (property "Value" "Q_PMOS_GSD" (id 1) (at 65.405 67.945 0)
+    (property "Value" "Q_PMOS_GSD" (id 1) (at 65.405 75.565 0)
       (effects (font (size 1.27 1.27)) (justify left))
     )
-    (property "Footprint" "Package_TO_SOT_SMD:SOT-23-3" (id 2) (at 76.2 69.215 0)
+    (property "Footprint" "Package_TO_SOT_SMD:SOT-23-3" (id 2) (at 76.2 74.295 0)
       (effects (font (size 1.27 1.27)) hide)
     )
@@
     (pin "1")
   )
-  (symbol (lib_id "Device:Q_PMOS_GSD") (at 111.125 116.205 0) (unit 1)
+  (symbol (lib_id "Device:Q_PMOS_GSD") (at 111.125 116.205 0) (mirror x) (unit 1)
     (in_bom yes) (on_board yes)
     (property "Reference" "Q18" (id 0) (at 116.205 116.205 0)
       (effects (font (size 1.27 1.27)) (justify left))
     )
-    (property "Value" "Q_PMOS_GSD" (id 1) (at 105.41 112.395 0)
+    (property "Value" "Q_PMOS_GSD" (id 1) (at 105.41 120.015 0)
       (effects (font (size 1.27 1.27)) (justify left))
     )
-    (property "Footprint" "Package_TO_SOT_SMD:SOT-23-3" (id 2) (at 116.205 113.665 0)
+    (property "Footprint" "Package_TO_SOT_SMD:SOT-23-3" (id 2) (at 116.205 118.745 0)
       (effects (font (size 1.27 1.27)) hide)
     )
